Commit message: fix oritation cam

File: husky_description/urdf/decorations.urdf.xacro (robot description, xacro)
@@ -152,5 +152,5 @@
           <parent link="base_link" />
           <child link="top_plate_link"/>
-          <origin xyz="0.0812 0 0.245" rpy="0 0 0"/>
+          <origin xyz="-0.0812 0 0.245" rpy="0 0 0"/>
         </joint>
         <!-- Top plate front link -->

File: husky_description/urdf/husky_macro.urdf.xacro (robot description, xacro)
@@ -125,5 +125,6 @@
     <xacro:if value="${topbar_needed_realsense}">
       <xacro:sensor_arch prefix="" parent="top_plate_link">
-        <origin xyz="-0.35 0 0.51" rpy="0 0 -3.14" />
+        <!-- <origin xyz="-0.35 0 0.51" rpy="0 0 -3.14" /> -->
+        <origin xyz="0.35 0 0.51" rpy="0 0 0" />
       </xacro:sensor_arch>
     </xacro:if>
