Commit message: update camera

File: husky_description/urdf/accessories/d435_mount.urdf.xacro (robot description, xacro)
@@ -3,75 +3,8 @@
   <!-- params: parent, xyz, rpy -->
   <xacro:macro name="d435_mount" params="parent xyz:='0.02 0 0.015' rpy:='0 0 0'">
-    <!-- ① rigid frame where the plugin attaches -->
-    <link name="realsense_link" />
-    <joint name="realsense_joint" type="fixed">
-      <parent link="${parent}" />
-      <child link="realsense_link" />
+    <xacro:include filename="$(find realsense2_description)/urdf/_d435.urdf.xacro" />
+    <xacro:sensor_d435 name="camera" topics_ns="camera" parent="${parent}" publish_pointcloud="true">
       <origin xyz="${xyz}" rpy="${rpy}" />
-    </joint>
-    <!-- ② visual mesh so you see the camera in RViz -->
-    <link name="realsense_link_visual" self_collide="0">
-      <visual>
-        <origin xyz="0 0 0" rpy="-1.57 0 -1.57" />
-        <geometry>
-          <!-- <mesh filename="package://realsense2_description/meshes/sensors/d435.dae" scale="1 1
-          1" /> -->
-          <!-- <mesh filename="package://realsense2_description/meshes/d435.dae" scale="1 1 1"/> -->
-          <!-- <mesh filename="package://husky_assets/meshes/d435.dae" scale="1 1 1" /> -->
-          <!-- <mesh filename="package://husky_assets/meshes/d435.dae" />-->
-          <mesh filename="package://husky_description/meshes/accessories/d435.dae" />
-        </geometry>
-        <material name="white" />
-      </visual>
-    </link>
-    <joint name="realsense_visual_joint" type="fixed">
-      <parent link="realsense_link" />
-      <child link="realsense_link_visual" />
-    </joint>
-    <!-- ③ the Gazebo plugin block straight from the repo README -->
-    <gazebo reference="realsense_link">
-      <gravity>0</gravity>
-      <sensor name="cameracolor" type="camera">
-        <camera name="camera">
-          <horizontal_fov>1.57</horizontal_fov>
-          <image>
-            <width>1280</width>
-            <height>720</height>
-            <format>RGB_INT8</format>
-          </image>
-          <clip>
-            <near>0.1</near>
-            <far>100</far>
-          </clip>
-        </camera>
-        <always_on>1</always_on>
-        <update_rate>30</update_rate>
-        <visualize>1</visualize>
-      </sensor>
-      <sensor name="cameradepth" type="depth">
-        <camera name="camera">
-          <horizontal_fov>1.57</horizontal_fov>
-          <image>
-            <width>1280</width>
-            <height>720</height>
-          </image>
-          <clip>
-            <near>0.1</near>
-            <far>100</far>
-          </clip>
-        </camera>
-        <always_on>1</always_on>
-        <update_rate>30</update_rate>
-        <visualize>0</visualize>
-      </sensor>
-      <!-- ⚠ Point-cloud can crash Gazebo; start false & re-enable later -->
-      <plugin name="camera" filename="librealsense_gazebo_plugin.so">
-        <prefix>camera</prefix>
-        <depthUpdateRate>30</depthUpdateRate>
-        <colorUpdateRate>30</colorUpdateRate>
-        <infraredUpdateRate>1</infraredUpdateRate>
-        <pointCloud>false</pointCloud>  <!-- default true -->
-      </plugin>
-    </gazebo>
+    </xacro:sensor_d435>
   </xacro:macro>
 </robot>
